File: GR8RAM.sch (KiCad schematic (older format))
At the start: 69 parts, among them J1 AppleIIBus, J2 JTAG, J4 JTAG, J5 JTAG, SW1 FW, U1 EPM240T100C5N, U13 25M, U14 74LVC1G125GW, U16 74LVC1G125GW, U2 W9825, U3 W25Q128JVSIQ, U4 74AHC245PW, U5 74AHC245PW, U6 74AHC245PW, U8 XC6206P332MR, U9 74AHC245PW

Commit message: Finished SRAM design schematic
Parts:
- removed J2, J5: JTAG, Connector:Tag-Connect_TC2050-IDC-FP_2x05_P1.27mm_Vertical, symbol Connector_Generic:Conn_02x05_Odd_Even
- removed J4: JTAG, Connector_IDC:IDC-Header_2x05_P2.54mm_Vertical, symbol Connector_Generic:Conn_02x05_Odd_Even
- removed R22, R31: 33, stdpads:R_0603, symbol Device:R_Small
- removed R28, R29: 22k, stdpads:R_0603, symbol Device:R_Small
- removed RN1, RN2, RN3: 4x33, stdpads:R4_0402, symbol Device:R_Pack04
- removed RN5: 4x10k, stdpads:R4_0402, symbol Device:R_Pack04
- removed SW1: FW, stdpads:SW_DIP_SPSTx02_Slide_DSHP02TS_P1.27mm, symbol Switch:SW_DIP_x02
- removed U1: EPM240T100C5N, stdpads:TQFP-100_14x14mm_P0.5mm, symbol GW_PLD:EPM240T100
- removed U13: 25M, stdpads:Crystal_SMD_3225-4Pin_3.2x2.5mm, symbol GW_Logic:Oscillator_4P
- removed U14, U16: 74LVC1G125GW, stdpads:SOT-353, symbol GW_Logic:741G125GW
- removed U2: W9825, stdpads:TSOP-II-54_22.2x10.16mm_P0.8mm, symbol GW_RAM:SDRAM-16Mx16-TSOP2-54
- removed U3: W25Q128JVSIQ, stdpads:SOIC-8_5.3mm, symbol GW_RAM:SPIFlash-SO-8
- removed U4, U5, U9: 74AHC245PW, stdpads:TSSOP-20_4.4x6.5mm_P0.65mm, symbol GW_Logic:74245
- removed U8: XC6206P332MR, stdpads:SOT-23, symbol GW_Power:AP2125
- added BT?: CR2032, symbol Device:Battery_Cell
- added D? (x2): 1N5819, symbol Device:D_Schottky_Small_ALT
- added Q?: MMBT3904, Package_TO_SOT_SMD:SOT-23, symbol Transistor_BJT:MMBT3904
- added R? (x2): 10k, symbol Device:R_Small
- added U1, U13, U27, U36, U44, U55: 74LVC86APW, stdpads:TSSOP-14_4.4x5mm_P0.65mm, symbol 74xx:74LS86
- added U10, U21, U30, U43, U49, U59: 74LVC257APW, stdpads:TSSOP-16_4.4x5mm_P0.65mm, symbol GW_Logic:74257
- added U11, U14, U15, U16, U19, U2, U20, U22, U23, U24, U25, U26, U28, U29, U3, U31, U32, U33, U34, U35, U37, U38, U4, U5, U50, U56, U62, U63, U7, U8, U9: 74LVC08APW, stdpads:TSSOP-14_4.4x5mm_P0.65mm, symbol 74xx:74LS08
- added U12: 74LVC32APW, stdpads:TSSOP-14_4.4x5mm_P0.65mm, symbol 74xx:74LS32
- added U17, U39, U52: 74LVC273PW, stdpads:TSSOP-20_4.4x6.5mm_P0.65mm, symbol GW_Logic:74273
- added U18, U40, U53: 74AHC245PW, stdpads:TSSOP-20_4.4x6.5mm_P0.65mm, symbol GW_Logic:74245
- added U41, U42: SRAM-512Kx16-TSOP2-44, stdpads:TSOP-II-44_400mil_P0.8mm, symbol GW_RAM:SRAM-512Kx16-TSOP2-44
- added U45, U46, U57, U58, U61: 74LVC138APW, stdpads:TSSOP-16_4.4x5mm_P0.65mm, symbol GW_Logic:74138
- added U47, U51, U54, U60: 74LVC04APW, stdpads:TSSOP-14_4.4x5mm_P0.65mm, symbol 74xx:74LS04
- added U48: 74LVC74APW, stdpads:TSSOP-14_4.4x5mm_P0.65mm, symbol 74xx:74LS74
Connections:
- net labels added: AD0, AD1, AD2, AD3, AD4, AD5, AD6, AD7, ALSEL, AMSEL, AQ0, AQ1, AQ10, AQ11, AQ12, AQ13, AQ14, AQ15, AQ16, AQ17, AQ18, AQ19, AQ2, AQ20, AQ21, AQ22, AQ23, AQ3, AQ4, AQ5, AQ6, AQ7, AQ8, AQ9, B0, DSEL, D~OE~, I0, I1, I10, I11, I12, I13, I14, I15, I16, I17, I18, I19, I2, I20, I21, I22, I23, I3, I4, I5, I6, I7, I8, I9, IOEN, R~CS~, T0, T1, T10, T11, T12, T13, T14, T15, T16, T17, T18, T19, T2, T20, T21, T22, T23, T3, T4, T5, T6, T7, T8, T9, VBAT, ~AHRD~, ~AHWR~, ~ALRD~, ~ALWR~, ~AMRD~, ~AMWR~, ~B0~, ~D16~, ~D7~, ~DRD~, ~DSEL~, ~DWR~, ~IOEN~, ~R0L~, ~R0U~, ~R1L~, ~R1U~, ~R2L~, ~R2U~, ~R3L~, ~R3U~, ~WE~
- net labels removed: ACLK, Dr0, Dr1, Dr2, Dr3, Dr4, Dr5, Dr6, Dr7, FCK, FD2, FD3, FW0, FW1, F~CS~, MISO, MOSI, RA0, RA1, RA10, RA11, RA12, RA13, RA14, RA15, RA2, RA3, RA4, RA5, RA6, RA7, RA8, RA9, RCLK, RES~OE~, RPHI0, RR~W~in, R~DEVSEL~, R~IOSEL~, R~IOSTRB~, R~RES~, SA0, SA1, SA10, SA11, SA12, SA2, SA3, SA4, SA5, SA6, SA7, SA8, SA9, SBA0, SBA1, SCKE, SD0, SD1, SD2, SD3, SD4, SD5, SD6, SD7, SDQMH, SDQML, S~CAS~, S~CS~, S~RAS~, S~WE~, TCK, TDI, TDO, TMS
- wire segments 209 -> 776
- no-connect marks 16 -> 0
Other:
- moved on the sheet: C1, C10, C11, C12, C13, C14, C15, C16, C18, C19, C2, C20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
